Commit message: fixed bugs of pyrr

File: urdf_examples/estun/estun.urdf (robot description, URDF)
Before this commit: robot ER10-900, 7 links, 6 joints
Links:
- link 1_Link: geometry collision mesh filename=meshes/1_Link.STL; visual mesh filename=meshes/1_Link.STL
- link 2_Link: geometry collision mesh filename=meshes/2_Link.STL; visual mesh filename=meshes/2_Link.STL
- link 3_Link: geometry collision mesh filename=meshes/3_Link.STL; visual mesh filename=meshes/3_Link.STL
- link 4_Link: geometry collision mesh filename=meshes/4_Link.STL; visual mesh filename=meshes/4_Link.STL
- link 5_Link: geometry collision mesh filename=meshes/5_Link.STL; visual mesh filename=meshes/5_Link.STL
- link 6_Link: geometry collision mesh filename=meshes/6_Link.STL; visual mesh filename=meshes/6_Link.STL
- link base_link: geometry collision mesh filename=meshes/base_link.STL; visual mesh filename=meshes/base_link.STL
