Commit message: fixed MDH, kinematics code gen, add requirements

File: urdf_examples/half_exo/half_exo.urdf (robot description, URDF)
Before this commit: robot exo, 4 links, 3 joints
Joints:
- joint R_hip_ab: limit lower=0 upper=0 effort=0 velocity=0 -> effort=1000 velocity=10
- joint R_hip_flex: limit lower=0 upper=0 effort=0 velocity=0 -> effort=1000 velocity=10
- joint R_knee: limit lower=0 upper=0 effort=0 velocity=0 -> effort=1000 velocity=10
