Commit message: revise urdf of drop

File: urdf_examples/drop/robot.urdf (robot description, URDF)
Before this commit: robot Robot, 4 links, 3 joints
Joints:
- joint first_Jiont: limit lower=0 upper=0 effort=0 velocity=0 -> effort=1000 velocity=10
- joint second_Jiont: limit lower=0 upper=0 effort=0 velocity=0 -> effort=1000 velocity=10
- joint third_Joint: limit lower=0 upper=0 effort=0 velocity=0 -> effort=1000 velocity=10

Commit message: Update robot.urdf

File: urdf_examples/drop/robot.urdf (robot description, URDF)
Before this commit: robot Robot, 4 links, 3 joints
Joints:
- removed joint first_Jiont
- removed joint second_Jiont
- added joint first_Joint: type revolute, parent base_link, child first_Link, origin xyz=0 0 0.1081 rpy=0 0 0, axis 0 0 1, limit effort=1000 velocity=10
- added joint second_Joint: type revolute, parent first_Link, child second_Link, origin xyz=0 0 0.045 rpy=1.5708 0 1.5798, axis 0 0 1, limit effort=1000 velocity=10
