Commit message: finished base para exporting and check code generation

File: urdf_examples/3r/urdf/3r.urdf (robot description, URDF)
Before this commit: robot 3r, 5 links, 4 joints
Links:
- link 1: geometry collision mesh filename=..\meshes\stl\base-Body.004.stl scale=1.0 1.0 1.0; visual mesh filename=..\meshes\stl\base-Body.004.stl scale=1.0 1.0 1.0
- link 2: geometry collision mesh filename=..\meshes\stl\arm-Body.005.stl scale=1.0 1.0 1.0; visual mesh filename=..\meshes\stl\arm-Body.005.stl scale=1.0 1.0 1.0
- link 3: geometry collision mesh filename=..\meshes\stl\arm2-Body.004.stl scale=1.0 1.0 1.0; visual mesh filename=..\meshes\stl\arm2-Body.004.stl scale=1.0 1.0 1.0
- link tool: geometry collision mesh filename=..\meshes\stl\tool-Body.stl scale=1.0 1.0 1.0; visual mesh filename=..\meshes\stl\tool-Body.stl scale=1.0 1.0 1.0
- link world: geometry collision mesh filename=..\meshes\stl\world-Body.003.stl scale=1.0 1.0 1.0; visual mesh filename=..\meshes\stl\world-Body.003.stl scale=1.0 1.0 1.0

File: urdf_examples/exo/exo.urdf (robot description, URDF)
Before this commit: robot exo, 7 links, 6 joints
Joints:
- joint L_hip_ab: limit lower=0 upper=0 effort=0 velocity=0 -> effort=100 velocity=10
- joint L_hip_flex: limit lower=0 upper=0 effort=0 velocity=0 -> effort=100 velocity=10
- joint L_knee: limit lower=0 upper=0 effort=0 velocity=0 -> effort=100 velocity=10
- joint R_hip_ab: limit lower=0 upper=0 effort=0 velocity=0 -> effort=100 velocity=10
- joint R_hip_flex: limit lower=0 upper=0 effort=0 velocity=0 -> effort=100 velocity=10
- joint R_knee: limit lower=0 upper=0 effort=0 velocity=0 -> effort=100 velocity=10

Commit message: update invdyn_baseparams with symengine

File: urdf_examples/3r/urdf/3r.urdf (robot description, URDF)
Before this commit: robot 3r, 5 links, 4 joints
Links:
- link 1: geometry collision mesh filename=../meshes/stl/base-Body.004.stl scale=1.0 1.0 1.0; visual mesh filename=../meshes/stl/base-Body.004.stl scale=1.0 1.0 1.0
- link 2: geometry collision mesh filename=../meshes/stl/arm-Body.005.stl scale=1.0 1.0 1.0; visual mesh filename=../meshes/stl/arm-Body.005.stl scale=1.0 1.0 1.0
- link 3: geometry collision mesh filename=../meshes/stl/arm2-Body.004.stl scale=1.0 1.0 1.0; visual mesh filename=../meshes/stl/arm2-Body.004.stl scale=1.0 1.0 1.0
- link tool: geometry collision mesh filename=../meshes/stl/tool-Body.stl scale=1.0 1.0 1.0; visual mesh filename=../meshes/stl/tool-Body.stl scale=1.0 1.0 1.0
- link world: geometry collision mesh filename=../meshes/stl/world-Body.003.stl scale=1.0 1.0 1.0; visual mesh filename=../meshes/stl/world-Body.003.stl scale=1.0 1.0 1.0
